File: 65HE_V2_PCB/Switches.kicad_sch (KiCad schematic)
At the start: 136 parts

Commit message: placed switches and muxes
Parts:
- removed HE68: SW_MX_HE, PCM_marbastlib-xp-he:SW_MX_HE_90deg_1u, symbol PCM_marbastlib-he:SW_MX_HE
- removed HE_C68: 100nF, Capacitor_SMD:C_0805_2012Metric, symbol Device:C_Small
- added MUX1, MUX2, MUX3, MUX4, MUX5, MUX6, MUX7, MUX8, MUX9: SN74LV4051A, Package_SO:TSSOP-16_4.4x5mm_P0.65mm, symbol 4xxx:4051
- added MUX_C1, MUX_C2, MUX_C3, MUX_C4, MUX_C5, MUX_C6, MUX_C7, MUX_C8, MUX_C9: 100nF, Capacitor_SMD:C_0805_2012Metric, symbol Device:C_Small
- added S1: MX_stab, PCM_marbastlib-mx:STAB_MX_2u, symbol PCM_marbastlib-mx:MX_stab
- added S2, S3: MX_stab, PCM_marbastlib-mx:STAB_MX_2.25u, symbol PCM_marbastlib-mx:MX_stab
- added S4: MX_stab, PCM_marbastlib-mx:STAB_MX_6.25u, symbol PCM_marbastlib-mx:MX_stab
Connections:
- net +3.3VA: now also MUX1.16 (VDD), MUX2.16 (VDD), MUX3.16 (VDD), MUX4.16 (VDD), MUX5.16 (VDD), MUX6.16 (VDD), MUX7.16 (VDD), MUX8.16 (VDD), MUX9.16 (VDD), MUX_C1.2, MUX_C2.2, MUX_C3.2, MUX_C4.2, MUX_C5.2, MUX_C6.2, MUX_C7.2, MUX_C8.2, MUX_C9.2
- net Earth: now also MUX1.6 (Inh), MUX1.7 (VEE), MUX1.8 (VSS), MUX2.6 (Inh), MUX2.7 (VEE), MUX2.8 (VSS), MUX3.6 (Inh), MUX3.7 (VEE), MUX3.8 (VSS), MUX4.6 (Inh), MUX4.7 (VEE), MUX4.8 (VSS), MUX5.6 (Inh), MUX5.7 (VEE), MUX5.8 (VSS), MUX6.6 (Inh), MUX6.7 (VEE), MUX6.8 (VSS), MUX7.6 (Inh), MUX7.7 (VEE), MUX7.8 (VSS), MUX8.6 (Inh), MUX8.7 (VEE), MUX8.8 (VSS), MUX9.6 (Inh), MUX9.7 (VEE), MUX9.8 (VSS), MUX_C1.1, MUX_C2.1, MUX_C3.1, MUX_C4.1, MUX_C5.1, MUX_C6.1, MUX_C7.1, MUX_C8.1, MUX_C9.1
- net HE1: no longer HE10.2 (VOUT), HE11.2 (VOUT), HE12.2 (VOUT), HE13.2 (VOUT), HE14.2 (VOUT), HE15.2 (VOUT), HE16.2 (VOUT), HE17.2 (VOUT), HE18.2 (VOUT), HE19.2 (VOUT), HE2.2 (VOUT), HE20.2 (VOUT), HE21.2 (VOUT), HE22.2 (VOUT), HE23.2 (VOUT), HE24.2 (VOUT), HE25.2 (VOUT), HE26.2 (VOUT), HE27.2 (VOUT), HE28.2 (VOUT), HE29.2 (VOUT), HE3.2 (VOUT), HE30.2 (VOUT), HE31.2 (VOUT), HE32.2 (VOUT), HE33.2 (VOUT), HE34.2 (VOUT), HE35.2 (VOUT), HE36.2 (VOUT), HE37.2 (VOUT), HE38.2 (VOUT), HE39.2 (VOUT), HE4.2 (VOUT), HE40.2 (VOUT), HE41.2 (VOUT), HE42.2 (VOUT), HE43.2 (VOUT), HE44.2 (VOUT), HE45.2 (VOUT), HE46.2 (VOUT), HE47.2 (VOUT), HE48.2 (VOUT), HE49.2 (VOUT), HE5.2 (VOUT), HE50.2 (VOUT), HE51.2 (VOUT), HE52.2 (VOUT), HE53.2 (VOUT), HE54.2 (VOUT), HE55.2 (VOUT), HE56.2 (VOUT), HE57.2 (VOUT), HE58.2 (VOUT), HE59.2 (VOUT), HE6.2 (VOUT), HE60.2 (VOUT), HE61.2 (VOUT), HE62.2 (VOUT), HE63.2 (VOUT), HE64.2 (VOUT), HE65.2 (VOUT), HE66.2 (VOUT), HE67.2 (VOUT), HE7.2 (VOUT), HE8.2 (VOUT), HE9.2 (VOUT)
- new net HE10: HE10.2 (VOUT)
- new net HE11: HE11.2 (VOUT)
- new net HE12: HE12.2 (VOUT)
- new net HE13: HE13.2 (VOUT)
- new net HE14: HE14.2 (VOUT)
- new net HE15: HE15.2 (VOUT)
- new net HE16: HE16.2 (VOUT)
- new net HE17: HE17.2 (VOUT)
- new net HE18: HE18.2 (VOUT)
- new net HE19: HE19.2 (VOUT)
- new net HE2: HE2.2 (VOUT)
- new net HE20: HE20.2 (VOUT)
- new net HE21: HE21.2 (VOUT)
- new net HE22: HE22.2 (VOUT)
- new net HE23: HE23.2 (VOUT)
- new net HE24: HE24.2 (VOUT)
- new net HE25: HE25.2 (VOUT)
- new net HE26: HE26.2 (VOUT)
- new net HE27: HE27.2 (VOUT)
- new net HE28: HE28.2 (VOUT)
- new net HE29: HE29.2 (VOUT)
- new net HE3: HE3.2 (VOUT)
- new net HE30: HE30.2 (VOUT)
- new net HE31: HE31.2 (VOUT)
- new net HE32: HE32.2 (VOUT)
- new net HE33: HE33.2 (VOUT)
- new net HE34: HE34.2 (VOUT)
- new net HE35: HE35.2 (VOUT)
- new net HE36: HE36.2 (VOUT)
- new net HE37: HE37.2 (VOUT)
- new net HE38: HE38.2 (VOUT)
- new net HE39: HE39.2 (VOUT)
- new net HE4: HE4.2 (VOUT)
- new net HE40: HE40.2 (VOUT)
- new net HE41: HE41.2 (VOUT)
- new net HE42: HE42.2 (VOUT)
- new net HE43: HE43.2 (VOUT)
- new net HE44: HE44.2 (VOUT)
- new net HE45: HE45.2 (VOUT)
- new net HE46: HE46.2 (VOUT)
- new net HE47: HE47.2 (VOUT)
- new net HE48: HE48.2 (VOUT)
- new net HE49: HE49.2 (VOUT)
- new net HE5: HE5.2 (VOUT)
- new net HE50: HE50.2 (VOUT)
- new net HE51: HE51.2 (VOUT)
- new net HE52: HE52.2 (VOUT)
- new net HE53: HE53.2 (VOUT)
- new net HE54: HE54.2 (VOUT)
- new net HE55: HE55.2 (VOUT)
- new net HE56: HE56.2 (VOUT)
- new net HE57: HE57.2 (VOUT)
- new net HE58: HE58.2 (VOUT)
- new net HE59: HE59.2 (VOUT)
- new net HE6: HE6.2 (VOUT)
- new net HE60: HE60.2 (VOUT)
- new net HE61: HE61.2 (VOUT)
- new net HE62: HE62.2 (VOUT)
- new net HE63: HE63.2 (VOUT)
- new net HE64: HE64.2 (VOUT)
- new net HE65: HE65.2 (VOUT)
- new net HE66: HE66.2 (VOUT)
- new net HE67: HE67.2 (VOUT)
- new net HE7: HE7.2 (VOUT)
- new net HE8: HE8.2 (VOUT)
- new net HE9: HE9.2 (VOUT)
- new net MUX1: MUX1.3 (X)
- new net MUX2: MUX2.3 (X)
- new net MUX3: MUX3.3 (X)
- new net MUX4: MUX4.3 (X)
- new net MUX5: MUX5.3 (X)
- new net MUX6: MUX6.3 (X)
- new net MUX7: MUX7.3 (X)
- new net MUX8: MUX8.3 (X)
- new net MUX9: MUX9.3 (X)
- new net Select1: MUX1.11 (A), MUX2.11 (A), MUX3.11 (A), MUX4.11 (A), MUX5.11 (A), MUX6.11 (A), MUX7.11 (A), MUX8.11 (A), MUX9.11 (A)
- new net Select2: MUX1.10 (B), MUX2.10 (B), MUX3.10 (B), MUX4.10 (B), MUX5.10 (B), MUX6.10 (B), MUX7.10 (B), MUX8.10 (B), MUX9.10 (B)
- new net Select3: MUX1.9 (C), MUX2.9 (C), MUX3.9 (C), MUX4.9 (C), MUX5.9 (C), MUX6.9 (C), MUX7.9 (C), MUX8.9 (C), MUX9.9 (C)
Other:
- moved on the sheet: HE64, HE65, HE66, HE67, HE_C64, HE_C65, HE_C66, HE_C67

Commit message: wired all the switched
Connections:
- net Earth: now also MUX4.12 (X3), MUX4.4 (X7)
- net HE1: now also MUX1.12 (X3)
- net HE10: now also MUX3.13 (X0)
- net HE11: now also MUX3.14 (X1)
- net HE12: now also MUX3.15 (X2)
- net HE13: now also MUX4.13 (X0)
- net HE14: now also MUX4.14 (X1)
- net HE15: now also MUX4.15 (X2)
- net HE16: now also MUX1.5 (X5)
- net HE17: now also MUX1.4 (X7)
- net HE18: now also MUX1.2 (X6)
- net HE19: now also MUX1.1 (X4)
- net HE2: now also MUX1.13 (X0)
- net HE20: now also MUX2.5 (X5)
- net HE21: now also MUX2.4 (X7)
- net HE22: now also MUX2.2 (X6)
- net HE23: now also MUX2.1 (X4)
- net HE24: now also MUX3.5 (X5)
- net HE25: now also MUX3.4 (X7)
- net HE26: now also MUX3.2 (X6)
- net HE27: now also MUX3.1 (X4)
- net HE28: now also MUX4.5 (X5)
- net HE29: now also MUX4.2 (X6)
- net HE3: now also MUX1.14 (X1)
- net HE30: now also MUX4.1 (X4)
- net HE31: now also MUX5.12 (X3)
- net HE32: now also MUX5.13 (X0)
- net HE33: now also MUX5.14 (X1)
- net HE34: now also MUX5.15 (X2)
- net HE35: now also MUX6.12 (X3)
- net HE36: now also MUX6.13 (X0)
- net HE37: now also MUX6.14 (X1)
- net HE38: now also MUX6.15 (X2)
- net HE39: now also MUX7.12 (X3)
- net HE4: now also MUX1.15 (X2)
- net HE40: now also MUX7.13 (X0)
- net HE41: now also MUX7.14 (X1)
- net HE42: now also MUX7.15 (X2)
- net HE43: now also MUX7.2 (X6)
- net HE44: now also MUX7.1 (X4)
- net HE45: now also MUX5.5 (X5)
- net HE46: now also MUX5.4 (X7)
- net HE47: now also MUX5.2 (X6)
- net HE48: now also MUX5.1 (X4)
- net HE49: now also MUX6.5 (X5)
- net HE5: now also MUX2.12 (X3)
- net HE50: now also MUX6.4 (X7)
- net HE51: now also MUX6.2 (X6)
- net HE52: now also MUX6.1 (X4)
- net HE53: now also MUX7.5 (X5)
- net HE54: now also MUX7.4 (X7)
- net HE55: now also MUX8.12 (X3)
- net HE56: now also MUX8.13 (X0)
- net HE57: now also MUX8.14 (X1)
- net HE58: now also MUX8.15 (X2)
- net HE59: now also MUX9.12 (X3)
- net HE6: now also MUX2.13 (X0)
- net HE60: now also MUX9.13 (X0)
- net HE61: now also MUX9.14 (X1)
- net HE62: now also MUX9.1 (X4)
- net HE63: now also MUX9.4 (X7)
- net HE64: now also MUX9.2 (X6)
- net HE65: now also MUX8.5 (X5)
- net HE66: now also MUX8.2 (X6)
- net HE67: now also MUX8.1 (X4)
- net HE7: now also MUX2.14 (X1)
- net HE8: now also MUX2.15 (X2)
- net HE9: now also MUX3.12 (X3)
