File: 65HE_V2_PCB/65HE_V2_PCB.kicad_pcb (KiCad board)
At the start: 2 copper layers, 1 part, among them U1 SW_MX_HE

Commit message: placed switches and muxes
Parts:
- added BOOT0: SW_SPST, PCM_marbastlib-various:SW_SPST_SKQG_WithStem, F.Cu at (485.6, 25.3)
- added C1: 100nF, Capacitor_SMD:C_0805_2012Metric, F.Cu at (468.8, 23.4)
- added C10: 10uF, Capacitor_SMD:C_1206_3216Metric, F.Cu at (493.2, 27.0)
- added C11: 10uF, Capacitor_SMD:C_1206_3216Metric, F.Cu at (493.2, 30.3)
- added C12: 10uF, Capacitor_SMD:C_1206_3216Metric, F.Cu at (493.2, 33.7)
- added C2: 100nF, Capacitor_SMD:C_0805_2012Metric, F.Cu at (468.8, 26.5)
- added C3: 100nF, Capacitor_SMD:C_0805_2012Metric, F.Cu at (468.8, 29.5)
- added C4: 100nF, Capacitor_SMD:C_0805_2012Metric, F.Cu at (468.8, 32.5)
- added C5: 100nF, Capacitor_SMD:C_0805_2012Metric, F.Cu at (468.8, 35.5)
- added C6: 100nF, Capacitor_SMD:C_0805_2012Metric, F.Cu at (468.8, 38.5)
- added C7: 100nF, Capacitor_SMD:C_0805_2012Metric, F.Cu at (468.8, 41.5)
- added C9: 10uF, Capacitor_SMD:C_1206_3216Metric, F.Cu at (493.2, 23.6)
- added D1: PRTR5V0U2X, Package_TO_SOT_SMD:SOT-143, F.Cu at (473.1, 48.6)
- added HE1: SW_MX_HE, PCM_marbastlib-xp-he:SW_MX_HE_90deg_1u, B.Cu at (79.0, 57.1)
- added HE10: SW_MX_HE, PCM_marbastlib-xp-he:SW_MX_HE_90deg_1u, B.Cu at (250.4, 57.1)
- added HE11: SW_MX_HE, PCM_marbastlib-xp-he:SW_MX_HE_90deg_1u, B.Cu at (269.5, 57.1)
- added HE12: SW_MX_HE, PCM_marbastlib-xp-he:SW_MX_HE_90deg_1u, B.Cu at (288.5, 57.1)
- added HE13: SW_MX_HE, PCM_marbastlib-xp-he:SW_MX_HE_90deg_1u, B.Cu at (307.6, 57.1)
- added HE14: SW_MX_HE, PCM_marbastlib-xp-he:SW_MX_HE_90deg_1u, B.Cu at (336.2, 57.1)
- added HE15: SW_MX_HE, PCM_marbastlib-xp-he:SW_MX_HE_90deg_1u, B.Cu at (364.7, 57.1)
- added HE16: SW_MX_HE, PCM_marbastlib-xp-he:SW_MX_HE_90deg_1u, B.Cu at (83.7, 76.2)
- added HE17: SW_MX_HE, PCM_marbastlib-xp-he:SW_MX_HE_90deg_1u, B.Cu at (107.6, 76.2)
- added HE18: SW_MX_HE, PCM_marbastlib-xp-he:SW_MX_HE_90deg_1u, B.Cu at (126.6, 76.2)
- added HE19: SW_MX_HE, PCM_marbastlib-xp-he:SW_MX_HE_90deg_1u, B.Cu at (145.7, 76.2)
- added HE2: SW_MX_HE, PCM_marbastlib-xp-he:SW_MX_HE_90deg_1u, B.Cu at (98.0, 57.1)
- added HE20: SW_MX_HE, PCM_marbastlib-xp-he:SW_MX_HE_90deg_1u, B.Cu at (164.7, 76.2)
- added HE21: SW_MX_HE, PCM_marbastlib-xp-he:SW_MX_HE_90deg_1u, B.Cu at (183.8, 76.2)
- added HE22: SW_MX_HE, PCM_marbastlib-xp-he:SW_MX_HE_90deg_1u, B.Cu at (202.8, 76.2)
- added HE23: SW_MX_HE, PCM_marbastlib-xp-he:SW_MX_HE_90deg_1u, B.Cu at (221.9, 76.2)
- added HE24: SW_MX_HE, PCM_marbastlib-xp-he:SW_MX_HE_90deg_1u, B.Cu at (240.9, 76.2)
- added HE25: SW_MX_HE, PCM_marbastlib-xp-he:SW_MX_HE_90deg_1u, B.Cu at (260.0, 76.2)
- added HE26: SW_MX_HE, PCM_marbastlib-xp-he:SW_MX_HE_90deg_1u, B.Cu at (279.0, 76.2)
- added HE27: SW_MX_HE, PCM_marbastlib-xp-he:SW_MX_HE_90deg_1u, B.Cu at (298.1, 76.2)
- added HE28: SW_MX_HE, PCM_marbastlib-xp-he:SW_MX_HE_90deg_1u, B.Cu at (317.1, 76.2)
- added HE29: SW_MX_HE, PCM_marbastlib-xp-he:SW_MX_HE_90deg_1u, B.Cu at (340.9, 76.2)
- added HE3: SW_MX_HE, PCM_marbastlib-xp-he:SW_MX_HE_90deg_1u, B.Cu at (117.1, 57.1)
- added HE30: SW_MX_HE, PCM_marbastlib-xp-he:SW_MX_HE_90deg_1u, B.Cu at (364.7, 76.2)
- added HE31: SW_MX_HE, PCM_marbastlib-xp-he:SW_MX_HE_90deg_1u, B.Cu at (86.1, 95.2)
- added HE32: SW_MX_HE, PCM_marbastlib-xp-he:SW_MX_HE_90deg_1u, B.Cu at (112.3, 95.2)
- added HE33: SW_MX_HE, PCM_marbastlib-xp-he:SW_MX_HE_90deg_1u, B.Cu at (131.4, 95.2)
- added HE34: SW_MX_HE, PCM_marbastlib-xp-he:SW_MX_HE_90deg_1u, B.Cu at (150.4, 95.2)
- added HE35: SW_MX_HE, PCM_marbastlib-xp-he:SW_MX_HE_90deg_1u, B.Cu at (169.5, 95.2)
- added HE36: SW_MX_HE, PCM_marbastlib-xp-he:SW_MX_HE_90deg_1u, B.Cu at (188.5, 95.2)
- added HE37: SW_MX_HE, PCM_marbastlib-xp-he:SW_MX_HE_90deg_1u, B.Cu at (207.6, 95.2)
- added HE38: SW_MX_HE, PCM_marbastlib-xp-he:SW_MX_HE_90deg_1u, B.Cu at (226.6, 95.2)
- added HE39: SW_MX_HE, PCM_marbastlib-xp-he:SW_MX_HE_90deg_1u, B.Cu at (245.7, 95.2)
- added HE4: SW_MX_HE, PCM_marbastlib-xp-he:SW_MX_HE_90deg_1u, B.Cu at (136.1, 57.1)
- added HE40: SW_MX_HE, PCM_marbastlib-xp-he:SW_MX_HE_90deg_1u, B.Cu at (264.7, 95.2)
- added HE41: SW_MX_HE, PCM_marbastlib-xp-he:SW_MX_HE_90deg_1u, B.Cu at (283.8, 95.2)
- added HE42: SW_MX_HE, PCM_marbastlib-xp-he:SW_MX_HE_90deg_1u, B.Cu at (302.8, 95.2)
- added HE43: SW_MX_HE, PCM_marbastlib-xp-he:SW_MX_HE_90deg_1u, B.Cu at (333.8, 95.2)
- added HE44: SW_MX_HE, PCM_marbastlib-xp-he:SW_MX_HE_90deg_1u, B.Cu at (364.7, 95.2)
- added HE45: SW_MX_HE, PCM_marbastlib-xp-he:SW_MX_HE_90deg_1u, B.Cu at (90.9, 114.3)
- added HE46: SW_MX_HE, PCM_marbastlib-xp-he:SW_MX_HE_90deg_1u, B.Cu at (121.8, 114.3)
- added HE47: SW_MX_HE, PCM_marbastlib-xp-he:SW_MX_HE_90deg_1u, B.Cu at (140.9, 114.3)
- added HE48: SW_MX_HE, PCM_marbastlib-xp-he:SW_MX_HE_90deg_1u, B.Cu at (159.9, 114.3)
- added HE49: SW_MX_HE, PCM_marbastlib-xp-he:SW_MX_HE_90deg_1u, B.Cu at (179.0, 114.3)
- added HE5: SW_MX_HE, PCM_marbastlib-xp-he:SW_MX_HE_90deg_1u, B.Cu at (155.2, 57.1)
- added HE50: SW_MX_HE, PCM_marbastlib-xp-he:SW_MX_HE_90deg_1u, B.Cu at (198.0, 114.3)
- added HE51: SW_MX_HE, PCM_marbastlib-xp-he:SW_MX_HE_90deg_1u, B.Cu at (217.1, 114.3)
- added HE52: SW_MX_HE, PCM_marbastlib-xp-he:SW_MX_HE_90deg_1u, B.Cu at (236.1, 114.3)
- added HE53: SW_MX_HE, PCM_marbastlib-xp-he:SW_MX_HE_90deg_1u, B.Cu at (255.2, 114.3)
- added HE54: SW_MX_HE, PCM_marbastlib-xp-he:SW_MX_HE_90deg_1u, B.Cu at (274.2, 114.3)
- added HE55: SW_MX_HE, PCM_marbastlib-xp-he:SW_MX_HE_90deg_1u, B.Cu at (293.3, 114.3)
- added HE56: SW_MX_HE, PCM_marbastlib-xp-he:SW_MX_HE_90deg_1u, B.Cu at (319.5, 114.3)
- added HE57: SW_MX_HE, PCM_marbastlib-xp-he:SW_MX_HE_90deg_1u, B.Cu at (345.7, 114.3)
- added HE58: SW_MX_HE, PCM_marbastlib-xp-he:SW_MX_HE_90deg_1u, B.Cu at (364.7, 114.3)
- added HE59: SW_MX_HE, PCM_marbastlib-xp-he:SW_MX_HE_90deg_1u, B.Cu at (81.4, 133.3)
- added HE6: SW_MX_HE, PCM_marbastlib-xp-he:SW_MX_HE_90deg_1u, B.Cu at (174.2, 57.1)
- added HE60: SW_MX_HE, PCM_marbastlib-xp-he:SW_MX_HE_90deg_1u, B.Cu at (105.2, 133.3)
- added HE61: SW_MX_HE, PCM_marbastlib-xp-he:SW_MX_HE_90deg_1u, B.Cu at (129.0, 133.3)
- added HE62: SW_MX_HE, PCM_marbastlib-xp-he:SW_MX_HE_90deg_1u, B.Cu at (200.4, 133.3)
- added HE63: SW_MX_HE, PCM_marbastlib-xp-he:SW_MX_HE_90deg_1u, B.Cu at (271.9, 133.3)
- added HE64: SW_MX_HE, PCM_marbastlib-xp-he:SW_MX_HE_90deg_1u, B.Cu at (295.7, 133.3)
- added HE65: SW_MX_HE, PCM_marbastlib-xp-he:SW_MX_HE_90deg_1u, B.Cu at (326.6, 133.3)
- added HE66: SW_MX_HE, PCM_marbastlib-xp-he:SW_MX_HE_90deg_1u, B.Cu at (345.7, 133.3)
- added HE67: SW_MX_HE, PCM_marbastlib-xp-he:SW_MX_HE_90deg_1u, B.Cu at (364.7, 133.3)
- added HE7: SW_MX_HE, PCM_marbastlib-xp-he:SW_MX_HE_90deg_1u, B.Cu at (193.3, 57.1)
- added HE8: SW_MX_HE, PCM_marbastlib-xp-he:SW_MX_HE_90deg_1u, B.Cu at (212.3, 57.1)
- added HE9: SW_MX_HE, PCM_marbastlib-xp-he:SW_MX_HE_90deg_1u, B.Cu at (231.4, 57.1)
- added HE_C1: 100nF, Capacitor_SMD:C_0805_2012Metric, B.Cu at (76.2, 57.1)
- added HE_C10: 100nF, Capacitor_SMD:C_0805_2012Metric, B.Cu at (247.7, 57.1)
- added HE_C11: 100nF, Capacitor_SMD:C_0805_2012Metric, B.Cu at (266.7, 57.1)
- added HE_C12: 100nF, Capacitor_SMD:C_0805_2012Metric, B.Cu at (285.8, 57.1)
- added HE_C13: 100nF, Capacitor_SMD:C_0805_2012Metric, B.Cu at (304.8, 57.1)
- added HE_C14: 100nF, Capacitor_SMD:C_0805_2012Metric, B.Cu at (333.4, 57.1)
- added HE_C15: 100nF, Capacitor_SMD:C_0805_2012Metric, B.Cu at (361.9, 57.1)
- added HE_C16: 100nF, Capacitor_SMD:C_0805_2012Metric, B.Cu at (81.0, 76.2)
- added HE_C17: 100nF, Capacitor_SMD:C_0805_2012Metric, B.Cu at (104.8, 76.2)
- added HE_C18: 100nF, Capacitor_SMD:C_0805_2012Metric, B.Cu at (123.8, 76.2)
- added HE_C19: 100nF, Capacitor_SMD:C_0805_2012Metric, B.Cu at (142.9, 76.2)
- added HE_C2: 100nF, Capacitor_SMD:C_0805_2012Metric, B.Cu at (95.2, 57.1)
- added HE_C20: 100nF, Capacitor_SMD:C_0805_2012Metric, B.Cu at (161.9, 76.2)
- added HE_C21: 100nF, Capacitor_SMD:C_0805_2012Metric, B.Cu at (181.0, 76.2)
- added HE_C22: 100nF, Capacitor_SMD:C_0805_2012Metric, B.Cu at (200.0, 76.2)
- added HE_C23: 100nF, Capacitor_SMD:C_0805_2012Metric, B.Cu at (219.1, 76.2)
- added HE_C24: 100nF, Capacitor_SMD:C_0805_2012Metric, B.Cu at (238.1, 76.2)
- added HE_C25: 100nF, Capacitor_SMD:C_0805_2012Metric, B.Cu at (257.2, 76.2)
- added HE_C26: 100nF, Capacitor_SMD:C_0805_2012Metric, B.Cu at (276.2, 76.2)
- added HE_C27: 100nF, Capacitor_SMD:C_0805_2012Metric, B.Cu at (295.3, 76.2)
- added HE_C28: 100nF, Capacitor_SMD:C_0805_2012Metric, B.Cu at (314.3, 76.2)
- added HE_C29: 100nF, Capacitor_SMD:C_0805_2012Metric, B.Cu at (338.1, 76.2)
- added HE_C3: 100nF, Capacitor_SMD:C_0805_2012Metric, B.Cu at (114.3, 57.1)
- added HE_C30: 100nF, Capacitor_SMD:C_0805_2012Metric, B.Cu at (361.9, 76.2)
- added HE_C31: 100nF, Capacitor_SMD:C_0805_2012Metric, B.Cu at (83.3, 95.2)
- added HE_C32: 100nF, Capacitor_SMD:C_0805_2012Metric, B.Cu at (109.5, 95.2)
- added HE_C33: 100nF, Capacitor_SMD:C_0805_2012Metric, B.Cu at (128.6, 95.2)
- added HE_C34: 100nF, Capacitor_SMD:C_0805_2012Metric, B.Cu at (147.6, 95.2)
- added HE_C35: 100nF, Capacitor_SMD:C_0805_2012Metric, B.Cu at (166.7, 95.2)
- added HE_C36: 100nF, Capacitor_SMD:C_0805_2012Metric, B.Cu at (185.7, 95.2)
- added HE_C37: 100nF, Capacitor_SMD:C_0805_2012Metric, B.Cu at (204.8, 95.2)
- added HE_C38: 100nF, Capacitor_SMD:C_0805_2012Metric, B.Cu at (223.8, 95.2)
- added HE_C39: 100nF, Capacitor_SMD:C_0805_2012Metric, B.Cu at (242.9, 95.2)
- added HE_C4: 100nF, Capacitor_SMD:C_0805_2012Metric, B.Cu at (133.3, 57.1)
- added HE_C40: 100nF, Capacitor_SMD:C_0805_2012Metric, B.Cu at (261.9, 95.2)
- added HE_C41: 100nF, Capacitor_SMD:C_0805_2012Metric, B.Cu at (281.0, 95.2)
- added HE_C42: 100nF, Capacitor_SMD:C_0805_2012Metric, B.Cu at (300.0, 95.2)
- added HE_C43: 100nF, Capacitor_SMD:C_0805_2012Metric, B.Cu at (331.0, 95.2)
- added HE_C44: 100nF, Capacitor_SMD:C_0805_2012Metric, B.Cu at (361.9, 95.2)
- added HE_C45: 100nF, Capacitor_SMD:C_0805_2012Metric, B.Cu at (88.1, 114.3)
- added HE_C46: 100nF, Capacitor_SMD:C_0805_2012Metric, B.Cu at (119.1, 114.3)
- added HE_C47: 100nF, Capacitor_SMD:C_0805_2012Metric, B.Cu at (138.1, 114.3)
- added HE_C48: 100nF, Capacitor_SMD:C_0805_2012Metric, B.Cu at (157.2, 114.3)
- added HE_C49: 100nF, Capacitor_SMD:C_0805_2012Metric, B.Cu at (176.2, 114.3)
- added HE_C5: 100nF, Capacitor_SMD:C_0805_2012Metric, B.Cu at (152.4, 57.1)
- added HE_C50: 100nF, Capacitor_SMD:C_0805_2012Metric, B.Cu at (195.3, 114.3)
- added HE_C51: 100nF, Capacitor_SMD:C_0805_2012Metric, B.Cu at (214.3, 114.3)
- added HE_C52: 100nF, Capacitor_SMD:C_0805_2012Metric, B.Cu at (233.4, 114.3)
- added HE_C53: 100nF, Capacitor_SMD:C_0805_2012Metric, B.Cu at (252.4, 114.3)
- added HE_C54: 100nF, Capacitor_SMD:C_0805_2012Metric, B.Cu at (271.5, 114.3)
- added HE_C55: 100nF, Capacitor_SMD:C_0805_2012Metric, B.Cu at (290.5, 114.3)
- added HE_C56: 100nF, Capacitor_SMD:C_0805_2012Metric, B.Cu at (316.7, 114.3)
- added HE_C57: 100nF, Capacitor_SMD:C_0805_2012Metric, B.Cu at (342.9, 114.3)
- added HE_C58: 100nF, Capacitor_SMD:C_0805_2012Metric, B.Cu at (361.9, 114.3)
- added HE_C59: 100nF, Capacitor_SMD:C_0805_2012Metric, B.Cu at (78.6, 133.3)
- added HE_C6: 100nF, Capacitor_SMD:C_0805_2012Metric, B.Cu at (171.4, 57.1)
- added HE_C60: 100nF, Capacitor_SMD:C_0805_2012Metric, B.Cu at (102.4, 133.3)
- added HE_C61: 100nF, Capacitor_SMD:C_0805_2012Metric, B.Cu at (126.2, 133.3)
- added HE_C62: 100nF, Capacitor_SMD:C_0805_2012Metric, B.Cu at (197.6, 133.3)
- added HE_C63: 100nF, Capacitor_SMD:C_0805_2012Metric, B.Cu at (269.1, 133.3)
- added HE_C64: 100nF, Capacitor_SMD:C_0805_2012Metric, B.Cu at (292.9, 133.3)
- added HE_C65: 100nF, Capacitor_SMD:C_0805_2012Metric, B.Cu at (323.9, 133.3)
- added HE_C66: 100nF, Capacitor_SMD:C_0805_2012Metric, B.Cu at (342.9, 133.3)
- added HE_C67: 100nF, Capacitor_SMD:C_0805_2012Metric, B.Cu at (361.9, 133.3)
- added HE_C7: 100nF, Capacitor_SMD:C_0805_2012Metric, B.Cu at (190.5, 57.1)
- added HE_C8: 100nF, Capacitor_SMD:C_0805_2012Metric, B.Cu at (209.6, 57.1)
- added HE_C9: 100nF, Capacitor_SMD:C_0805_2012Metric, B.Cu at (228.6, 57.1)
- added J1: Conn_01x04, Connector_JST:JST_SH_SM04B-SRSS-TB_1x04-1MP_P1.00mm_Horizontal, B.Cu at (136.0, 65.7)
- added MUX1: SN74LV4051A, Package_SO:TSSOP-16_4.4x5mm_P0.65mm, B.Cu at (112.3, 66.7)
- added MUX2: SN74LV4051A, Package_SO:TSSOP-16_4.4x5mm_P0.65mm, B.Cu at (188.5, 66.7)
- added MUX3: SN74LV4051A, Package_SO:TSSOP-16_4.4x5mm_P0.65mm, B.Cu at (264.7, 66.7)
- added MUX4: SN74LV4051A, Package_SO:TSSOP-16_4.4x5mm_P0.65mm, B.Cu at (333.4, 66.7)
- added MUX5: SN74LV4051A, Package_SO:TSSOP-16_4.4x5mm_P0.65mm, B.Cu at (126.6, 104.8)
- added MUX6: SN74LV4051A, Package_SO:TSSOP-16_4.4x5mm_P0.65mm, B.Cu at (202.8, 104.8)
- added MUX7: SN74LV4051A, Package_SO:TSSOP-16_4.4x5mm_P0.65mm, B.Cu at (278.6, 104.8)
- added MUX8: SN74LV4051A, Package_SO:TSSOP-16_4.4x5mm_P0.65mm, B.Cu at (336.2, 123.8)
- added MUX9: SN74LV4051A, Package_SO:TSSOP-16_4.4x5mm_P0.65mm, B.Cu at (178.2, 133.3)
- added MUX_C1: 100nF, Capacitor_SMD:C_0805_2012Metric, B.Cu at (460.0, 100.4)
- added MUX_C2: 100nF, Capacitor_SMD:C_0805_2012Metric, B.Cu at (460.0, 97.4)
- added MUX_C3: 100nF, Capacitor_SMD:C_0805_2012Metric, B.Cu at (460.0, 94.4)
- added MUX_C4: 100nF, Capacitor_SMD:C_0805_2012Metric, B.Cu at (460.0, 91.4)
- added MUX_C5: 100nF, Capacitor_SMD:C_0805_2012Metric, B.Cu at (460.0, 88.4)
- added MUX_C6: 100nF, Capacitor_SMD:C_0805_2012Metric, B.Cu at (460.0, 85.4)
- added MUX_C7: 100nF, Capacitor_SMD:C_0805_2012Metric, B.Cu at (460.0, 82.3)
- added MUX_C8: 100nF, Capacitor_SMD:C_0805_2012Metric, B.Cu at (460.0, 79.3)
- added MUX_C9: 100nF, Capacitor_SMD:C_0805_2012Metric, B.Cu at (460.0, 76.3)
- added NRST1: SW_SPST, PCM_marbastlib-various:SW_SPST_SKQG_WithStem, F.Cu at (485.6, 32.1)
- added R1: 5.1kΩ, Resistor_SMD:R_0805_2012Metric, F.Cu at (468.7, 44.5)
- added R2: 5.1kΩ, Resistor_SMD:R_0805_2012Metric, F.Cu at (468.7, 47.4)
- added S1: MX_stab, PCM_marbastlib-mx:STAB_MX_2u, F.Cu at (336.2, 57.1)
- added S2: MX_stab, PCM_marbastlib-mx:STAB_MX_2.25u, F.Cu at (333.8, 95.2)
- added S3: MX_stab, PCM_marbastlib-mx:STAB_MX_2.25u, F.Cu at (90.9, 114.3)
- added S4: MX_stab, PCM_marbastlib-mx:STAB_MX_6.25u, F.Cu at (200.4, 133.3)
- added U2: LD1117S33TR_SOT223, Package_TO_SOT_SMD:SOT-223-3_TabPin2, F.Cu at (475.9, 26.1)
- added U3: LD1117S33TR_SOT223, Package_TO_SOT_SMD:SOT-223-3_TabPin2, F.Cu at (475.9, 34.5)
- U1: value SW_MX_HE -> STM32F072CBTx; footprint PCM_marbastlib-xp-he:SW_MX_HE_0deg_1u -> Package_QFP:LQFP-48_7x7mm_P0.5mm
- moved U1 408.9 mm to (486.5, 41.1)
Connections:
- U1 pad 1: unconnected-(U1-VCC-Pad1) -> +3.3V
Other:
- board outline added: 303.8 x 94.2 mm

Commit message: Vega + Bakeneko Board Outline
Parts:
- U1: moved to B.Cu
- moved U1 428.4 mm to (61.5, 95.2)
Other:
- outline, holes or cut-outs redrawn

Commit message: holes for standoffs
Parts:
- added H1: M2, MountingHole:MountingHole_2.2mm_M2_Pad, F.Cu at (88.5, 57.1)
- added H2: M2, MountingHole:MountingHole_2.2mm_M2_Pad, F.Cu at (183.8, 57.1)
- added H3: M2, MountingHole:MountingHole_2.2mm_M2_Pad, F.Cu at (279.0, 57.1)
- added H4: M2, MountingHole:MountingHole_2.2mm_M2_Pad, F.Cu at (355.2, 66.7)
- added H5: M2, MountingHole:MountingHole_2.2mm_M2_Pad, F.Cu at (159.9, 85.7)
- added H6: M2, MountingHole:MountingHole_2.2mm_M2_Pad, F.Cu at (293.3, 85.7)
- added H7: M2, MountingHole:MountingHole_2.2mm_M2_Pad, F.Cu at (93.3, 133.3)
- added H8: M2, MountingHole:MountingHole_2.2mm_M2_Pad, F.Cu at (226.6, 123.8)
- added H9: M2, MountingHole:MountingHole_2.2mm_M2_Pad, F.Cu at (355.2, 133.3)
- moved HE_C11 5.56 mm to (272.3, 57.1), turned to 90 degrees
- moved HE_C15 5.56 mm to (367.5, 57.1), turned to 90 degrees
- moved HE_C43 5.56 mm to (336.6, 95.2), turned to 90 degrees
- moved HE_C44 5.56 mm to (367.5, 95.2), turned to 90 degrees
- moved HE_C55 5.56 mm to (296.1, 114.3), turned to 90 degrees
- moved HE_C57 5.56 mm to (348.5, 114.3), turned to 90 degrees
- moved HE_C58 5.56 mm to (367.5, 114.3), turned to 90 degrees
- moved HE_C10 5.56 mm to (253.2, 57.1), turned to 90 degrees
- moved HE_C2 5.56 mm to (100.8, 57.1), turned to 90 degrees
- moved HE_C3 5.56 mm to (119.9, 57.1), turned to 90 degrees
- moved HE_C31 5.56 mm to (88.9, 95.2), turned to 90 degrees
- moved HE_C32 5.56 mm to (115.1, 95.2), turned to 90 degrees
- moved HE_C33 5.56 mm to (134.1, 95.2), turned to 90 degrees
- moved HE_C34 5.56 mm to (153.2, 95.2), turned to 90 degrees
- moved HE_C35 5.56 mm to (172.2, 95.2), turned to 90 degrees
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
Commit message: wired all the switched
Parts:
- moved MUX_C1 344.8 mm to (117.1, 63.9), turned to 180 degrees
- moved MUX_C5 328.9 mm to (131.4, 102.0), turned to 180 degrees
- moved MUX_C8 288.8 mm to (174.2, 121.0), turned to 180 degrees
- moved MUX_C2 268.8 mm to (193.3, 63.9), turned to 180 degrees
- moved MUX_C6 253.0 mm to (207.6, 102.0), turned to 180 degrees
- moved MUX_C3 192.9 mm to (269.5, 63.9), turned to 180 degrees
- moved MUX_C7 177.7 mm to (283.4, 102.0), turned to 180 degrees
- moved MUX_C9 127.2 mm to (340.9, 121.0), turned to 180 degrees
- moved MUX_C4 124.9 mm to (338.1, 63.9), turned to 180 degrees
- moved MUX9 12.9 mm to (169.5, 123.8)
Connections:
- MUX1 pad 1: unconnected-(MUX1-X4-Pad1) -> HE19
- MUX1 pad 12: unconnected-(MUX1-X3-Pad12) -> HE1
- MUX1 pad 13: unconnected-(MUX1-X0-Pad13) -> HE2
- MUX1 pad 14: unconnected-(MUX1-X1-Pad14) -> HE3
- MUX1 pad 15: unconnected-(MUX1-X2-Pad15) -> HE4
- MUX1 pad 2: unconnected-(MUX1-X6-Pad2) -> HE18
- MUX1 pad 4: unconnected-(MUX1-X7-Pad4) -> HE17
- MUX1 pad 5: unconnected-(MUX1-X5-Pad5) -> HE16
- MUX2 pad 1: unconnected-(MUX2-X4-Pad1) -> HE23
- MUX2 pad 12: unconnected-(MUX2-X3-Pad12) -> HE5
- MUX2 pad 13: unconnected-(MUX2-X0-Pad13) -> HE6
- MUX2 pad 14: unconnected-(MUX2-X1-Pad14) -> HE7
- MUX2 pad 15: unconnected-(MUX2-X2-Pad15) -> HE8
- MUX2 pad 2: unconnected-(MUX2-X6-Pad2) -> HE22
- MUX2 pad 4: unconnected-(MUX2-X7-Pad4) -> HE21
- MUX2 pad 5: unconnected-(MUX2-X5-Pad5) -> HE20
- MUX3 pad 1: unconnected-(MUX3-X4-Pad1) -> HE27
- MUX3 pad 12: unconnected-(MUX3-X3-Pad12) -> HE9
- MUX3 pad 13: unconnected-(MUX3-X0-Pad13) -> HE10
- MUX3 pad 14: unconnected-(MUX3-X1-Pad14) -> HE11
- MUX3 pad 15: unconnected-(MUX3-X2-Pad15) -> HE12
- MUX3 pad 2: unconnected-(MUX3-X6-Pad2) -> HE26
- MUX3 pad 4: unconnected-(MUX3-X7-Pad4) -> HE25
- MUX3 pad 5: unconnected-(MUX3-X5-Pad5) -> HE24
- MUX4 pad 1: unconnected-(MUX4-X4-Pad1) -> HE30
- MUX4 pad 12: unconnected-(MUX4-X3-Pad12) -> Earth
- MUX4 pad 13: unconnected-(MUX4-X0-Pad13) -> HE13
- MUX4 pad 14: unconnected-(MUX4-X1-Pad14) -> HE14
- MUX4 pad 15: unconnected-(MUX4-X2-Pad15) -> HE15
- MUX4 pad 2: unconnected-(MUX4-X6-Pad2) -> HE29
- MUX4 pad 4: unconnected-(MUX4-X7-Pad4) -> Earth
- MUX4 pad 5: unconnected-(MUX4-X5-Pad5) -> HE28
- MUX5 pad 1: unconnected-(MUX5-X4-Pad1) -> HE48
- MUX5 pad 12: unconnected-(MUX5-X3-Pad12) -> HE31
- MUX5 pad 13: unconnected-(MUX5-X0-Pad13) -> HE32
- MUX5 pad 14: unconnected-(MUX5-X1-Pad14) -> HE33
- MUX5 pad 15: unconnected-(MUX5-X2-Pad15) -> HE34
- MUX5 pad 2: unconnected-(MUX5-X6-Pad2) -> HE47
- MUX5 pad 4: unconnected-(MUX5-X7-Pad4) -> HE46
- MUX5 pad 5: unconnected-(MUX5-X5-Pad5) -> HE45
- MUX6 pad 1: unconnected-(MUX6-X4-Pad1) -> HE52
- MUX6 pad 12: unconnected-(MUX6-X3-Pad12) -> HE35
- MUX6 pad 13: unconnected-(MUX6-X0-Pad13) -> HE36
- MUX6 pad 14: unconnected-(MUX6-X1-Pad14) -> HE37
- MUX6 pad 15: unconnected-(MUX6-X2-Pad15) -> HE38
- MUX6 pad 2: unconnected-(MUX6-X6-Pad2) -> HE51
- MUX6 pad 4: unconnected-(MUX6-X7-Pad4) -> HE50
- MUX6 pad 5: unconnected-(MUX6-X5-Pad5) -> HE49
- MUX7 pad 1: unconnected-(MUX7-X4-Pad1) -> HE44
- MUX7 pad 12: unconnected-(MUX7-X3-Pad12) -> HE39
- MUX7 pad 13: unconnected-(MUX7-X0-Pad13) -> HE40
- MUX7 pad 14: unconnected-(MUX7-X1-Pad14) -> HE41
- MUX7 pad 15: unconnected-(MUX7-X2-Pad15) -> HE42
- MUX7 pad 2: unconnected-(MUX7-X6-Pad2) -> HE43
- MUX7 pad 4: unconnected-(MUX7-X7-Pad4) -> HE54
- MUX7 pad 5: unconnected-(MUX7-X5-Pad5) -> HE53
- MUX8 pad 1: unconnected-(MUX8-X4-Pad1) -> HE67
- MUX8 pad 12: unconnected-(MUX8-X3-Pad12) -> HE55
- MUX8 pad 13: unconnected-(MUX8-X0-Pad13) -> HE56
- MUX8 pad 14: unconnected-(MUX8-X1-Pad14) -> HE57
- MUX8 pad 15: unconnected-(MUX8-X2-Pad15) -> HE58
- MUX8 pad 2: unconnected-(MUX8-X6-Pad2) -> HE66
- MUX8 pad 5: unconnected-(MUX8-X5-Pad5) -> HE65
- MUX9 pad 1: unconnected-(MUX9-X4-Pad1) -> HE62
- MUX9 pad 12: unconnected-(MUX9-X3-Pad12) -> HE59
- MUX9 pad 13: unconnected-(MUX9-X0-Pad13) -> HE60
- MUX9 pad 14: unconnected-(MUX9-X1-Pad14) -> HE61
- MUX9 pad 2: unconnected-(MUX9-X6-Pad2) -> HE64
- MUX9 pad 4: unconnected-(MUX9-X7-Pad4) -> HE63
Routing:
- net +3.3VA: track 0.00 -> 1646.9 mm, vias 0 -> 67
- net Select3: track 0.00 -> 518.4 mm, vias 0 -> 11
- net Select2: track 0.00 -> 513.2 mm, vias 0 -> 11
- net Select1: track 0.00 -> 508.6 mm, vias 0 -> 11
- net HE64: track 0.00 -> 131.0 mm, vias 0 -> 2
- net HE63: track 0.00 -> 109.1 mm, vias 0 -> 2
- net HE59: track 0.00 -> 96.0 mm, vias 0 -> 2
- net HE44: track 0.00 -> 94.2 mm, vias 0 -> 2
- net HE60: track 0.00 -> 72.2 mm, vias 0 -> 2
- net HE43: track 0.00 -> 63.6 mm, vias 0 -> 2
- net HE61: track 0.00 -> 49.2 mm, vias 0 -> 2
- net HE55: track 0.00 -> 49.1 mm, vias 0 -> 2
- net HE31: track 0.00 -> 46.7 mm, vias 0 -> 2
- net HE9: track 0.00 -> 39.6 mm, vias 0 -> 2
- net HE5: track 0.00 -> 39.6 mm, vias 0 -> 2
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- added copper zone on B.Cu, net Earth
- added copper zone on F.Cu, net Earth

Commit message: pcb done?
Parts:
- added SWD: TC2030, Connector:Tag-Connect_TC2030-IDC-FP_2x03_P1.27mm_Vertical, B.Cu at (81.4, 85.7)
- BOOT/RUN: renamed from BOOT0; footprint PCM_marbastlib-various:SW_SPST_SKQG_WithStem -> PCM_marbastlib-various:SW_MSK12C02-HB
- C1, C10, C11, C12, C2, C3, C4, C5, C6, C7, C9, D1, R1, R2, U2, U3: moved to B.Cu
- moved C10 382.4 mm to (114.7, 81.8), turned to 180 degrees
- moved C4 380.5 mm to (92.9, 91.3), turned to -90 degrees
- moved C5 379.9 mm to (91.7, 81.4), turned to 180 degrees
- moved C9 377.5 mm to (120.3, 81.8)
- moved C6 370.9 mm to (100.0, 78.2), turned to 90 degrees
- moved C12 370.5 mm to (125.8, 81.8), turned to 180 degrees
- moved C3 369.9 mm to (102.4, 80.6), turned to 90 degrees
- moved C7 365.6 mm to (106.0, 86.5)
- moved C11 365.5 mm to (131.4, 81.8)
- moved U2 363.7 mm to (117.5, 87.7), turned to -90 degrees
- moved U3 351.4 mm to (128.6, 87.7), turned to -90 degrees
- moved C1 338.9 mm to (133.3, 72.2), turned to 90 degrees
- moved D1 337.8 mm to (136.1, 72.6), turned to 180 degrees
- moved BOOT/RUN 274.9 mm to (233.0, 133.7), turned to 180 degrees
- moved RESET 264.2 mm to (241.7, 133.6), turned to -90 degrees
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- renumbered J1 to Connector, NRST1 to RESET
Connections:
- BOOT/RUN pad 1: +3.3V -> BOOT0
- BOOT/RUN pad 2: BOOT0 -> +3.3V
- D1 pad 2: D- -> D+
- D1 pad 3: D+ -> D-
- U1 pad 10: unconnected-(U1-PA0-Pad10) -> MUX1
- U1 pad 11: unconnected-(U1-PA1-Pad11) -> MUX4
- U1 pad 12: unconnected-(U1-PA2-Pad12) -> MUX8
- U1 pad 13: unconnected-(U1-PA3-Pad13) -> MUX3
- U1 pad 14: unconnected-(U1-PA4-Pad14) -> MUX2
- U1 pad 15: unconnected-(U1-PA5-Pad15) -> MUX5
- U1 pad 16: unconnected-(U1-PA6-Pad16) -> MUX9
- U1 pad 17: unconnected-(U1-PA7-Pad17) -> MUX6
- U1 pad 18: unconnected-(U1-PB0-Pad18) -> MUX7
Routing:
- net MUX8: track 0.00 -> 275.5 mm, vias 0 -> 2
- net MUX4: track 0.00 -> 246.1 mm, vias 0 -> 2
- net MUX7: track 0.00 -> 227.9 mm, vias 0 -> 2
- net BOOT0: track 0.00 -> 217.9 mm, vias 0 -> 3
- net +3.3V: track 0.00 -> 216.5 mm, vias 0 -> 3
- net NRST: track 0.00 -> 209.8 mm, vias 0 -> 5
- net +3.3VA: track 1646.9 -> 1835.8 mm, vias 67 -> 73
- net MUX3: track 0.00 -> 188.4 mm, vias 0 -> 2
- net MUX6: track 0.00 -> 151.8 mm, vias 0 -> 2
- net MUX9: track 0.00 -> 145.8 mm, vias 0 -> 2
- net MUX2: track 0.00 -> 114.2 mm, vias 0 -> 2
- net D-: track 0.00 -> 74.8 mm, vias 0 -> 2
- net D+: track 0.00 -> 73.4 mm, vias 0 -> 2
- net MUX5: track 0.00 -> 73.2 mm, vias 0 -> 2
- net +5V: track 0.00 -> 46.6 mm, vias 0 -> 2
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