File: 65HE_V2_PCB/65HE_V2_PCB.kicad_sch (KiCad schematic)
At the start: 20 parts, among them J1 Conn_01x04, U1 STM32F072CBTx, U2 LD1117S33TR_SOT223, U3 LD1117S33TR_SOT223

Commit message: holes for standoffs
Parts:
- added H1, H2, H3, H4, H5, H6, H7, H8, H9: M2, MountingHole:MountingHole_2.2mm_M2_Pad, symbol Mechanical:MountingHole_Pad
Connections:
- no-connect marks 0 -> 9

Commit message: pcb done?
Parts:
- added J2: TC2030, Connector:Tag-Connect_TC2030-IDC-FP_2x03_P1.27mm_Vertical, symbol Connector:Conn_ARM_SWD_TagConnect_TC2030
- BOOT0: footprint PCM_marbastlib-various:SW_SPST_SKQG_WithStem -> PCM_marbastlib-various:SW_MSK12C02-HB
Connections:
- net +3.3V: now also BOOT0.2 (B), J2.1 (VCC); no longer BOOT0.1 (A)
- net BOOT0: now also BOOT0.1 (A); no longer BOOT0.2 (B)
- net D+: now also D1.2 (I/O1); no longer D1.3 (I/O2)
- net D-: now also D1.3 (I/O2); no longer D1.2 (I/O1)
- net Earth: now also J2.5 (GND)
- net NRST: now also J2.3 (~{RESET})
- net SWCLK: now also J2.4 (SWCLK)
- net SWDIO: now also J2.2 (SWDIO)
- net MUX1: now reaches U1.10 (PA0)
- net MUX4: now reaches U1.11 (PA1)
- net MUX8: now reaches U1.12 (PA2)
- net MUX3: now reaches U1.13 (PA3)
- net MUX2: now reaches U1.14 (PA4)
- net MUX5: now reaches U1.15 (PA5)
- net MUX9: now reaches U1.16 (PA6)
- net MUX6: now reaches U1.17 (PA7)
- net MUX7: now reaches U1.18 (PB0)
- no-connect marks 9 -> 10
